Commit message: large untracked commit

File: src/seven_robot_description/urdf/wheel.urdf.xacro (robot description, xacro)
@@ -55,5 +55,5 @@
 			</collision>
 		</link>
-		<joint name=" ${prefix}_joint" type="continuous">
+		<joint name="${prefix}_joint" type="continuous">
 			<parent link="base_link"/>
 			<child link=" ${prefix}_link"/>
