Commit message: urdf.launch now works. fixed the mesh scale for robot_base and wheel

File: src/seven_robot_description/urdf/robot.urdf.xacro (robot description, xacro)
@@ -34,9 +34,11 @@
 ****************************************************************************/
 -->
-<robot name="seven" xmlns:xacro="http://wiki.ros.org/wiki/xacro">
+<robot name="seven" xmlns:xacro="http://www.ros.org/wiki/xacro">
 	<xacro:property name="PI" value="3.14159"/>
 	<xacro:include filename="$(find seven_robot_description)/urdf/wheel.urdf.xacro"/>
 	<xacro:include filename="$(find seven_robot_description)/urdf/sick.urdf.xacro"/>
-	<!--robot base dimensions: includes the top enclosure size and bearing size-->
+	<xacro:arg name="robot_namespace" default="/" />
+	<!--robot base dimensions: includes the top enclosure
+			and flange bearing offsets-->
 	<xacro:property name="base_size_x" value="0.6307"/>
 	<xacro:property name="base_size_y" value="0.5285"/>
@@ -52,17 +54,18 @@
 			<origin rpy="0 0 0" xyz="0 0 0"/>
 			<geometry>
-				<mesh filename="package://seven_robot_descripiton/meshes/robot_base.dae"/>
+				<mesh filename="package://seven_robot_description/meshes/robot_base.dae"/>
 			</geometry>
 		</visual>
 		<collision>
-		<origin xyz="0 0 0" rpy="0 0 0">
+		<origin xyz="0 0 0" rpy="0 0 0"/>
 		<geometry>
-		<box size="${base_x_size + sick_mount_offset} ${base_size_y} ${base_size_z}">
+			<box size="${base_size_x + sick_collision_offset} ${base_size_y} ${base_size_z}"/>
 		</geometry>
 		</collision>
 	</link>
 	<link name="base_footprint"/>
+	<!--This is the footprint of our base which lies on the ground at all times-->
 	<joint name="base_footprint_joint" type="fixed">
-		<origin xyz="0 0 ${wheel_vertical_offset} - ${wheel_radius}" rpy="0 0 0"/>
+		<origin xyz="0 0 ${wheel_vertical_offset - wheel_radius}" rpy="0 0 0"/>
 		<parent link="base_link"/>
 		<child link="base_footprint"/>
@@ -80,16 +83,31 @@
 		<child link="inertial_link"/>
 	</joint>
+	<link name="imu_link">
+	</link>
+	<joint name="base_imu_joint" type="fixed">
+		<origin xyz="0 0 0" rpy="0 0 0"/>
+		<parent link="base_link"/>
+		<child link="imu_link"/>
+	</joint>
+	<link name="camera">
+	</link>
+	<joint name="base_camera_joint" type="fixed">
+		<origin xyz="0 0 0" rpy="0 0 0"/>
+		<parent link="base_link"/>
+		<child link="camera"/>
+	</joint>
+	<xacro:sick prefix="mirror_origin"/>
 	<!--wheel macros-->
-	<xacro:seven_wheel wheel_prefix="front_right">
-		<origin xyz="${wheel_base}/2 -${track_length/2 + wheel_width} ${wheel_vertical_offset}" rpy="0 0 0"/>
+	<xacro:seven_wheel prefix="frontRight">
+		<origin xyz="${wheel_base/2} -${track_length/2 + wheel_width} ${wheel_vertical_offset}" rpy="${PI/2} 0 0"/>
 	</xacro:seven_wheel>
-	<xacro:seven_wheel wheel_prefix="rear_right">
-		<origin xyz="-${wheel_base}/2 -${track_length/2 + wheel_width} ${wheel_vertical_offset}" rpy="0 0 0"/>
+	<xacro:seven_wheel prefix="rearRight">
+		<origin xyz="-${wheel_base/2} -${track_length/2 + wheel_width} ${wheel_vertical_offset}" rpy="${PI/2} 0 0"/>
 	</xacro:seven_wheel>
-	<xacro:seven_wheel wheel_prefix="front_left">
-		<origin xyz="${wheel_base}/2 ${track_length/2 + wheel_width} ${wheel_vertical_offset}" rpy="0 0 0"/>
+	<xacro:seven_wheel prefix="frontLeft">
+		<origin xyz="${wheel_base/2} ${track_length/2 + wheel_width} ${wheel_vertical_offset}" rpy="-${PI/2} 0 0"/>
 	</xacro:seven_wheel>
-	<xacro:seven_wheel wheel_prefix="rear_left">
-		<origin xyz="-${wheel_base}/2 ${track_length/2 + wheel_width} ${wheel_vertical_offset}" rpy="0 0 0"/>
+	<xacro:seven_wheel prefix="rearLeft">
+		<origin xyz="-${wheel_base/2} ${track_length/2 + wheel_width} ${wheel_vertical_offset}" rpy="-${PI/2} 0 0"/>
 	</xacro:seven_wheel>
 </robot>

File: src/seven_robot_description/urdf/sick.urdf.xacro (robot description, xacro)
@@ -34,5 +34,13 @@
 ****************************************************************************/
 -->
-<robot name="sick_lms2xx" xmlns:xacro="http:wiki.ros.org/wiki/xacro">
-	<xacro:property name="sick_mount_offset" value="0.1611"/>
+<robot name="sick_lms2xx" xmlns:xacro="http://www.ros.org/wiki/xacro">
+	<xacro:property name="sick_collision_offset" value="0.1611"/>
+	<xacro:macro name="sick" params="prefix">
+		<link name="${prefix}_link"/>
+		<joint name="base_${prefix}_joint" type="fixed">
+			<origin xyz="0.3739 0 0.0980" rpy="0 0 0"/>
+			<parent link="base_link"/>
+			<child link="${prefix}_link"/>
+		</joint>
+	</xacro:macro>
 </robot>

File: src/seven_robot_description/urdf/wheel.urdf.xacro (robot description, xacro)
@@ -34,7 +34,7 @@
 ****************************************************************************/
 -->
-<robot xmlns:xacro="http://www.wiki.ros.org/wiki/xacro" name="seven_wheel">
-	<xacro:macro name="seven_wheel" params="wheel_prefix *joint_pose">
-		<link name="${wheel_prefix}_wheel_link">
+<robot xmlns:xacro="http://www.ros.org/wiki/xacro" name="seven_wheel">
+	<xacro:macro name="seven_wheel" params="*joint_pose prefix">
+		<link name=" ${prefix}_link">
 			<inertial>
 				<mass value="1.900"/>
@@ -49,22 +49,22 @@
 			</visual>
 			<collision>
-				<origin xyz="0 0 0" rpy="0 0 0"/>
+				<origin xyz="0 0 0" rpy="${PI/2} 0 0"/>
 				<geometry>
-			 		<cylinder radius="${wheel_radius}" length="${wheel_length}"/>
+			 		<cylinder radius="${wheel_radius}" length="${wheel_width}"/>
 				</geometry>
 			</collision>
 		</link>
-		<joint name="${wheel_prefix}_joint" type="continuous">
+		<joint name=" ${prefix}_joint" type="continuous">
 			<parent link="base_link"/>
-			<child link="$(wheel_prefix)_wheel_link"/>
+			<child link=" ${prefix}_link"/>
 			<xacro:insert_block name="joint_pose"/>
-			<axis xyz="0 1 0" rpy="0 0 0">
+			<axis xyz="0 0 1" rpy="0 0 0"/>
 		</joint>
-		<transmission name="${wheel_prefix}_wheeltrans" type="SimpleTransmission">
+		<transmission name=" ${prefix}_wheeltrans" type="SimpleTransmission">
 			<type>transmission_interface/SimpleTransmission</type>
-			<actuator name="${wheel_prefix}_motor">
+			<actuator name=" ${prefix}_motor">
 				<mechanicalReduction>2</mechanicalReduction>
 			</actuator>
-			<joint name="${wheel_prefix}_joint">
+			<joint name="$${prefix}_joint">
 				<hardwareInterface>hardware_interface/VelocityJointInterface</hardwareInterface>
 			</joint>

Commit message: added sick_lms link and imu_link

File: src/seven_robot_description/urdf/robot.urdf.xacro (robot description, xacro)
@@ -35,4 +35,7 @@
 -->
 <robot name="seven" xmlns:xacro="http://www.ros.org/wiki/xacro">
+	<xacro:arg name="laser_enabled" default="FALSE"/>
+	<xacro:arg name="laser_xyz" default="$(optenv SEVEN_LMS2XX_XYZ 0.2750 0.0 0.1267)"/>
+	<xacro:arg name="laser_rpy" default="$(optenv SEVEN_LMS2XX_RPY 0.0 0.0 0.0)"/>
 	<xacro:property name="PI" value="3.14159"/>
 	<xacro:include filename="$(find seven_robot_description)/urdf/wheel.urdf.xacro"/>
@@ -52,5 +55,5 @@
 	<link name="base_link">
 		<visual>
-			<origin rpy="0 0 0" xyz="0 0 0"/>
+			<origin rpy="0 0 ${PI}" xyz="0 0 0"/>
 			<geometry>
 				<mesh filename="package://seven_robot_description/meshes/robot_base.dae"/>
@@ -58,7 +61,7 @@
 		</visual>
 		<collision>
-		<origin xyz="0 0 0" rpy="0 0 0"/>
+		<origin xyz="0 0 ${base_size_z/2}" rpy="0 0 0"/>
 		<geometry>
-			<box size="${base_size_x + sick_collision_offset} ${base_size_y} ${base_size_z}"/>
+			<box size="${base_size_x} ${base_size_y} ${base_size_z}"/>
 		</geometry>
 		</collision>
@@ -86,5 +89,5 @@
 	</link>
 	<joint name="base_imu_joint" type="fixed">
-		<origin xyz="0 0 0" rpy="0 0 0"/>
+		<origin xyz="0 0 0.250" rpy="0 0 0"/>
 		<parent link="base_link"/>
 		<child link="imu_link"/>
@@ -97,5 +100,4 @@
 		<child link="camera"/>
 	</joint>
-	<xacro:sick prefix="mirror_origin"/>
 	<!--wheel macros-->
 	<xacro:seven_wheel prefix="frontRight">
@@ -111,3 +113,6 @@
 		<origin xyz="-${wheel_base/2} ${track_length/2 + wheel_width} ${wheel_vertical_offset}" rpy="-${PI/2} 0 0"/>
 	</xacro:seven_wheel>
+	<xacro:sick_mount prefix="base">
+			<origin xyz="$(arg laser_xyz)" rpy="$(arg laser_rpy)"/>
+	</xacro:sick_mount>
 </robot>

File: src/seven_robot_description/urdf/sick.urdf.xacro (robot description, xacro)
@@ -35,11 +35,35 @@
 -->
 <robot name="sick_lms2xx" xmlns:xacro="http://www.ros.org/wiki/xacro">
-	<xacro:property name="sick_collision_offset" value="0.1611"/>
-	<xacro:macro name="sick" params="prefix">
-		<link name="${prefix}_link"/>
-		<joint name="base_${prefix}_joint" type="fixed">
-			<origin xyz="0.3739 0 0.0980" rpy="0 0 0"/>
-			<parent link="base_link"/>
-			<child link="${prefix}_link"/>
+	<xacro:macro name="sick_mount" params="prefix *joint_pose">
+		<link name="${prefix}_sick_link">
+			<inertial>
+				<mass value="4.12"/>
+				<origin xyz="0 0 0" rpy="0 0 0"/>
+				<inertia ixx="0" ixy="0" ixz="0" iyy="0" iyz="0" izz="0"/>
+			</inertial>
+			<visual>
+				<origin xyz="0 0 0" rpy="0 0 ${PI}"/>
+				<geometry>
+					<mesh filename="package://seven_robot_description/meshes/sick.dae"/>
+				</geometry>
+			</visual>
+			<collision>
+				<origin xyz="0 0 0" rpy="0 0 0"/>
+				<geometry>
+					<box size="0.155 0.156 .210"/>
+				</geometry>
+			</collision>
+		</link>
+		<joint name="${prefix}_sick_joint" type="fixed">
+			<parent link="${prefix}_link"/>
+			<child link="${prefix}_sick_link"/>
+			<xacro:insert_block name="joint_pose"/>
+		</joint>
+		<link name="laser_head"/>
+		<!--joint between the sensor body origin and laser head-->
+		<joint name="laser_head_joint" type="fixed">
+			<origin xyz="0.0930 0 -0.0295" rpy="0 0 0"/>
+			<parent link="${prefix}_sick_link"/>
+			<child link="laser_head"/>
 		</joint>
 	</xacro:macro>

Commit message: align robot imu_link with NED

File: src/seven_robot_description/urdf/robot.urdf.xacro (robot description, xacro)
@@ -89,5 +89,5 @@
 	</link>
 	<joint name="base_imu_joint" type="fixed">
-		<origin xyz="0 0 0.250" rpy="0 0 0"/>
+		<origin xyz="0 0 0.250" rpy="${PI} 0 0"/>
 		<parent link="base_link"/>
 		<child link="imu_link"/>

Commit message: Y axis of imu inverted not Z

File: src/seven_robot_description/urdf/robot.urdf.xacro (robot description, xacro)
@@ -55,5 +55,5 @@
 	<link name="base_link">
 		<visual>
-			<origin rpy="0 0 ${PI}" xyz="0 0 0"/>
+						<origin rpy="0 0 ${PI}" xyz="0 0 0"/>
 			<geometry>
 				<mesh filename="package://seven_robot_description/meshes/robot_base.dae"/>

Commit message: fix params and launch file formats. imu_link fixed in urdf

File: src/seven_robot_description/urdf/robot.urdf.xacro (robot description, xacro)
@@ -89,5 +89,5 @@
 	</link>
 	<joint name="base_imu_joint" type="fixed">
-		<origin xyz="0 0 0.250" rpy="${PI} 0 0"/>
+		<origin xyz="0 0 0.250" rpy="0 0 0"/>
 		<parent link="base_link"/>
 		<child link="imu_link"/>

Commit message: fix urdf and changes to ekf params

File: src/seven_robot_description/urdf/robot.urdf.xacro (robot description, xacro)
@@ -50,10 +50,10 @@
 	<xacro:property name="wheel_base" value="0.3440"/>
 	<xacro:property name="track_length" value="0.5366"/>
-	<xacro:property name="wheel_vertical_offset" value="0.07"/>
+	<xacro:property name="wheel_vertical_offset" value="0.12"/>
 	<xacro:property name="wheel_width" value="0.08"/>
 	<xacro:property name="wheel_radius" value="0.130"/>
 	<link name="base_link">
 		<visual>
-						<origin rpy="0 0 ${PI}" xyz="0 0 0"/>
+			<origin rpy="0 0 ${PI}" xyz="0 0 0.05"/>
 			<geometry>
 				<mesh filename="package://seven_robot_description/meshes/robot_base.dae"/>
@@ -93,10 +93,10 @@
 		<child link="imu_link"/>
 	</joint>
-	<link name="camera">
+	<link name="camera_link">
 	</link>
 	<joint name="base_camera_joint" type="fixed">
-		<origin xyz="0 0 0" rpy="0 0 0"/>
+		<origin xyz="0.4335 0 0.272" rpy="0 0 0"/>
 		<parent link="base_link"/>
-		<child link="camera"/>
+		<child link="camera_link"/>
 	</joint>
 	<!--wheel macros-->
