Commit message: fixed robot description

File: src/seven_robot_description/urdf/pu_wheel.urdf.xacro (robot description, xacro)
@@ -43,5 +43,5 @@
 			</inertial>
 			<visual>
-				<origin xyz="0 0 0" rpy="${PI/2} 0 0"/>
+				<origin xyz="0 0 0" rpy="0 0 0"/>
 				<geometry>
 					<mesh filename="package://seven_robot_description/meshes/PU_WHEEL.dae"/>
@@ -49,5 +49,5 @@
 			</visual>
 			<collision>
-				<origin xyz="0 0 0" rpy="${PI/2} 0 0"/>
+				<origin xyz="0 0 0" rpy="0 0 0"/>
 				<geometry>
 			 		<cylinder radius="${wheel_radius}" length="${wheel_width}"/>

File: src/seven_robot_description/urdf/sr-100.urdf.xacro (robot description, xacro)
@@ -112,5 +112,5 @@
 	</xacro:pu_wheel>
 	<xacro:pu_wheel prefix="Left">
-		<origin xyz="-0.0013 0.33014 0.04280" rpy="-${PI/2} 0 0"/>
+		<origin xyz="-0.0013 0.33014 0.04280" rpy="${-PI/2} 0 0"/>
 	</xacro:pu_wheel>
 	<xacro:sick_lms_1xx name="sick" ros_topic="scan"/>

Commit message: fix inertia matrix

File: src/seven_robot_description/urdf/pu_wheel.urdf.xacro (robot description, xacro)
@@ -59,5 +59,10 @@
 			<child link=" ${prefix}_link"/>
 			<xacro:insert_block name="joint_pose"/>
-			<axis xyz="0 0 1" rpy="0 0 0"/>
+			<xacro:if value="${prefix == 'Right'}">
+				<axis xyz="0 0 -1" rpy="0 0 0"/>
+			</xacro:if>
+			<xacro:if value="${prefix == 'Left'}">
+			 <axis xyz="0 0 1" rpy="0 0 0"/>
+			</xacro:if>
 		</joint>
 		<transmission name=" ${prefix}_wheeltrans" type="SimpleTransmission">

File: src/seven_robot_description/urdf/sr-100.urdf.xacro (robot description, xacro)
@@ -37,4 +37,5 @@
 	<xacro:property name="PI" value="3.14159"/>
   <xacro:arg name="use_nominal_extrinsics" default="false"/>
+	<xacro:include filename="$(find seven_robot_description)/urdf/sr-100.gazebo"/>
 	<xacro:include filename="$(find seven_robot_description)/urdf/pu_wheel.urdf.xacro"/>
 	<xacro:include filename="$(find seven_robot_description)/urdf/_d415.urdf.xacro"/>
@@ -60,8 +61,8 @@
 		</visual>
 		<collision>
-		<origin xyz="0 0 0" rpy="0 0 0"/>
-		<geometry>
-			<box size="${base_size_x} ${base_size_y} ${base_size_z}"/>
-		</geometry>
+		 <origin xyz="0 0 0.204528" rpy="0 0 0"/>
+		 <geometry>
+			<box size="${base_size_x} ${base_size_y} 0.47057"/>
+		 </geometry>
 		</collision>
 	</link>
@@ -75,6 +76,6 @@
 		<inertial>
 			<mass value="47.4"/>
-			<origin xyz="-0.001443 -0.000133 0.1181" rpy="0 0 0"/>
-			<inertia ixx="1.9397" ixy="-0.0051" ixz="0.0803" iyx="-0.0051" iyy="2.3585" iyz="0.0107" izx="0.0803" izy="0.0107" izz="2.2906"/>
+			<origin xyz="-0.01687 -0.00816 0.37647" rpy="0 0 0"/>
+			<inertia ixx="12585" ixy="-15.56" ixz="536.42" iyx="-15.56" iyy="806.894" iyz="-130.895" izx="-536.424" izy="-130.895" izz="5242.6"/>
 		</inertial>
 	</link>
