Commit message: fix sr-100 urdf

File: src/seven_robot_description/urdf/sr-100.urdf.xacro (robot description, xacro)
@@ -92,5 +92,5 @@
 	</joint>
 	<joint name="sick_base_joint" type="fixed">
-	 <origin xyz="0.41121 -0.31152 0.38036" rpy="${PI} 0.0 ${PI/4}"/>
+	 <origin xyz="0.41121 -0.31152 0.38036" rpy="${PI} 0.0 ${-PI/4}"/>
    <parent link="base_link"/>
 	 <child link="sick_mount_link"/>

Commit message: minor changes

File: src/seven_robot_description/urdf/sr-100.urdf.xacro (robot description, xacro)
@@ -92,5 +92,5 @@
 	</joint>
 	<joint name="sick_base_joint" type="fixed">
-	 <origin xyz="0.41121 -0.31152 0.38036" rpy="${PI} 0.0 ${-PI/4}"/>
+	 <origin xyz="0.41121 -0.31152 0.18972" rpy="${PI} 0.0 ${-PI/4}"/>
    <parent link="base_link"/>
 	 <child link="sick_mount_link"/>
@@ -116,5 +116,5 @@
 	<xacro:sick_lms_1xx name="sick" ros_topic="scan"/>
 	<xacro:sensor_d415 parent="base_link" use_nominal_extrinsics="$(arg use_nominal_extrinsics)">
-		<origin xyz="0.44215 0.005 0.38036" rpy="0 0 0"/>
+		<origin xyz="0.42720 0.005 0.36786" rpy="0 0 0"/>
 	</xacro:sensor_d415>
 	<xacro:sonarMount parent="base_link" name="sonarArrayMount">

Commit message: minor

File: src/seven_robot_description/urdf/sr-100.urdf.xacro (robot description, xacro)
@@ -112,5 +112,5 @@
 	</xacro:pu_wheel>
 	<xacro:pu_wheel prefix="Left">
-		<origin xyz="-0.0013 0.33014 0.04280" rpy="${-PI/2} 0 0"/>
+		<origin xyz="-0.0013 0.33014 0.04280" rpy="-${PI/2} 0 0"/>
 	</xacro:pu_wheel>
 	<xacro:sick_lms_1xx name="sick" ros_topic="scan"/>

Commit message: fix sr-100 urdf and add gazebo sims

File: src/seven_robot_description/urdf/sr-100.urdf.xacro (robot description, xacro)
@@ -40,4 +40,5 @@
 	<xacro:include filename="$(find seven_robot_description)/urdf/pu_wheel.urdf.xacro"/>
 	<xacro:include filename="$(find seven_robot_description)/urdf/_d415.urdf.xacro"/>
+	<xacro:include filename="$(find seven_robot_description)/urdf/_d415.gazebo.xacro"/>
 	<xacro:include filename="$(find seven_robot_description)/urdf/sick_lms1xx.urdf.xacro"/>
 	<xacro:include filename="$(find seven_robot_description)/urdf/caster_wheel.urdf.xacro"/>
@@ -45,4 +46,5 @@
 	<xacro:include filename="$(find seven_robot_description)/urdf/sonar.urdf.xacro"/>
 	<xacro:arg name="robot_namespace" default="/" />
+	<xacro:arg name="camera_name" default="sensor_d415"/>
 	<xacro:property name="base_size_x" value="0.97923"/>
 	<xacro:property name="base_size_y" value="0.77916"/>
@@ -92,10 +94,30 @@
 		<child link="imu_link"/>
 	</joint>
+  <gazebo reference="imu_link">
+	 <gravity>true</gravity>
+	 <sensor name="adis_imu" type="imu">
+	  <always_on>true</always_on>
+		<update_rate>100</update_rate>
+		<visualize>true</visualize>
+		<topic>__default_topic__</topic>
+		<plugin filename="libgazebo_ros_imu_sensor.so" name="imu_plugin">
+		 <topicName>imu</topicName>
+		 <bodyName>imu_link</bodyName>
+		 <updateRateHz>100</updateRateHz>
+		 <gaussianNoise>0</gaussianNoise>
+		 <xyzOffset>0 0 0</xyzOffset>
+		 <rpyOffset>0 0 0</rpyOffset>
+		 <frameName>imu_link</frameName>
+		 <initialOrientationAsReference>false</initialOrientationAsReference>
+		</plugin>
+		 <pose>0 0 0 0 0 0</pose>
+	 </sensor>
+	</gazebo>
 	<joint name="sick_base_joint" type="fixed">
-	 <origin xyz="0.41121 -0.31152 0.38036" rpy="${PI} 0.0 ${-PI/4}"/>
+	 <origin xyz="0.41121 -0.31152 0.18972" rpy="${PI} 0.0 ${-PI/4}"/>
    <parent link="base_link"/>
 	 <child link="sick_mount_link"/>
 	</joint>
-	<xacro:caster_wheel prefix="frontRight">
+ 	<xacro:caster_wheel prefix="frontRight">
 		<origin xyz="0.35015 -0.24985 0.10687" rpy="0 0 0"/>
 	</xacro:caster_wheel>
@@ -116,7 +138,8 @@
 	</xacro:pu_wheel>
 	<xacro:sick_lms_1xx name="sick" ros_topic="scan"/>
-	<xacro:sensor_d415 parent="base_link" use_nominal_extrinsics="$(arg use_nominal_extrinsics)">
-		<origin xyz="0.44215 0.005 0.38036" rpy="0 0 0"/>
+	<xacro:sensor_d415 parent="base_link" name="$(arg camera_name)" use_nominal_extrinsics="$(arg use_nominal_extrinsics)">
+		<origin xyz="0.42720 0.005 0.36786" rpy="0 0 0"/>
 	</xacro:sensor_d415>
+	<xacro:gazebo_d435 camera_name="$(arg camera_name)" reference_link="$(arg camera_name)_link" topics_ns="/" depth_optical_frame="$(arg camera_name)_depth_optical_frame" color_optical_frame="$(arg camera_name)_color_optical_frame" infrared1_optical_frame="$(arg camera_name)_infrared1_optical_frame" infrared2_optical_frame="$(arg camera_name)_infrared2_optical_frame"/>
 	<xacro:sonarMount parent="base_link">
     <origin xyz="0.42915 -0.00015 0.06192" rpy="0 0 0"/>
