Commit message: urdf changes updated for the second model

File: src/seven_robot_description/urdf/_d415.gazebo.xacro (robot description, xacro)
@@ -13,5 +13,4 @@
       <enable_wind>0</enable_wind>
       <kinematic>0</kinematic>
-      <gravity>1</gravity>
       <!--<mu>1</mu>-->
       <mu2>1</mu2>

File: src/seven_robot_description/urdf/robot.urdf.xacro (robot description, xacro)
@@ -44,13 +44,13 @@
 	<!--robot base dimensions: includes the top enclosure
 			and flange bearing offsets-->
-	<xacro:property name="base_size_x" value="0.6307"/>
-	<xacro:property name="base_size_y" value="0.5285"/>
-	<xacro:property name="base_size_z" value="0.3305"/>
+	<xacro:property name="base_size_x" value="0.820"/>
+	<xacro:property name="base_size_y" value="0.550"/>
+	<xacro:property name="base_size_z" value="0.358"/>
 	<!--wheel mounting includes offsets induced by bearings-->
-	<xacro:property name="wheel_base" value="0.3440"/>
+	<xacro:property name="wheel_base" value="0.387"/>
 	<xacro:property name="track_length" value="0.5366"/>
-	<xacro:property name="wheel_vertical_offset" value="0.12"/>
-	<xacro:property name="wheel_width" value="0.08"/>
-	<xacro:property name="wheel_radius" value="0.130"/>
+	<xacro:property name="wheel_vertical_offset" value="0.03736"/>
+	<xacro:property name="wheel_width" value="0.07"/>
+	<xacro:property name="wheel_radius" value="0.08641"/>
 	<link name="base_link">
 		<visual>

Commit message: RPM Ping commit

File: src/seven_robot_description/urdf/_d415.gazebo.xacro (robot description, xacro)
@@ -113,24 +113,24 @@
       <plugin name="${topics_ns}" filename="librealsense_gazebo_plugin.so">
         <prefix>${camera_name}</prefix>
-      	<depthUpdateRate>60.0</depthUpdateRate>
-      	<colorUpdateRate>60.0</colorUpdateRate>
-      	<infraredUpdateRate>60.0</infraredUpdateRate>
-      	<depthTopicName>depth/image_raw</depthTopicName>
-      	<depthCameraInfoTopicName>depth/camera_info</depthCameraInfoTopicName>
-      	<colorTopicName>color/image_raw</colorTopicName>
-      	<colorCameraInfoTopicName>color/camera_info</colorCameraInfoTopicName>
-      	<infrared1TopicName>infra1/image_raw</infrared1TopicName>
-      	<infrared1CameraInfoTopicName>infra1/camera_info</infrared1CameraInfoTopicName>
-      	<infrared2TopicName>infra2/image_raw</infrared2TopicName>
-      	<infrared2CameraInfoTopicName>infra2/camera_info</infrared2CameraInfoTopicName>
-      	<colorOpticalframeName>${color_optical_frame}</colorOpticalframeName>
-      	<depthOpticalframeName>${depth_optical_frame}</depthOpticalframeName>
-      	<infrared1OpticalframeName>${infrared1_optical_frame}</infrared1OpticalframeName>
-      	<infrared2OpticalframeName>${infrared2_optical_frame}</infrared2OpticalframeName>
-      	<rangeMinDepth>0.2</rangeMinDepth>
-      	<rangeMaxDepth>10.0</rangeMaxDepth>
-      	<pointCloud>false</pointCloud>
-      	<pointCloudTopicName>depth/points</pointCloudTopicName>
-      	<pointCloudCutoff>0.5</pointCloudCutoff>
+      	<depthUpdateRate>${camera_name}/60.0</depthUpdateRate>
+      	<colorUpdateRate>${camera_name}/60.0</colorUpdateRate>
+      	<infraredUpdateRate>${camera_name}/60.0</infraredUpdateRate>
+      	<depthTopicName>${camera_name}/depth/image_raw</depthTopicName>
+      	<depthCameraInfoTopicName>${camera_name}/depth/camera_info</depthCameraInfoTopicName>
+      	<colorTopicName>${camera_name}/color/image_raw</colorTopicName>
+      	<colorCameraInfoTopicName>${camera_name}/color/camera_info</colorCameraInfoTopicName>
+      	<infrared1TopicName>${camera_name}/infra1/image_raw</infrared1TopicName>
+      	<infrared1CameraInfoTopicName>${camera_name}/infra1/camera_info</infrared1CameraInfoTopicName>
+      	<infrared2TopicName>${camera_name}/infra2/image_raw</infrared2TopicName>
+      	<infrared2CameraInfoTopicName>${camera_name}/infra2/camera_info</infrared2CameraInfoTopicName>
+      	<colorOpticalframeName>${camera_name}/${color_optical_frame}</colorOpticalframeName>
+      	<depthOpticalframeName>${camera_name}/${depth_optical_frame}</depthOpticalframeName>
+      	<infrared1OpticalframeName>${camera_name}/${infrared1_optical_frame}</infrared1OpticalframeName>
+      	<infrared2OpticalframeName>${camera_name}/${infrared2_optical_frame}</infrared2OpticalframeName>
+      	<rangeMinDepth>${camera_name}/0.2</rangeMinDepth>
+      	<rangeMaxDepth>${camera_name}/10.0</rangeMaxDepth>
+      	<pointCloud>${camera_name}/false</pointCloud>
+      	<pointCloudTopicName>${camera_name}/depth/points</pointCloudTopicName>
+      	<pointCloudCutoff>${camera_name}/0.5</pointCloudCutoff>
       </plugin>
     </gazebo>

File: src/seven_robot_description/urdf/sr-300.urdf.xacro (robot description, xacro)
@@ -59,5 +59,5 @@
 	<link name="base_link">
     <visual>
-			<origin rpy="0 0 0" xyz="0 0 0"/>
+			<origin rpy="${PI} 0 0" xyz="0 0 0"/>
 			<geometry>
 				<mesh filename="package://seven_robot_description/meshes/sr300_chasis.dae"/>
@@ -111,5 +111,5 @@
   </gazebo>
 	<joint name="sick_base_joint" type="fixed">
-	 <origin xyz="0.3661 0.2171 -0.13329" rpy="0 0 ${PI/4}"/>
+		<origin xyz="0.375 -0.219 0.13329" rpy="${PI} 0 -${PI/4}"/>
    <parent link="base_link"/>
 	 <child link="sick_mount_link"/>
@@ -123,8 +123,8 @@
 	<xacro:sick_lms_1xx name="sick" ros_topic="scan"/>
 	<xacro:sensor_d415_left parent="base_link" name="$(arg camera_name_left)" use_nominal_extrinsics="$(arg use_nominal_extrinsics)">
-		<origin xyz="0.42 0.09026 -0.03433" rpy="-1.5140654 0.2588659 -0.032099"/>
+		<origin xyz="0.415 0.1178 0.022233" rpy="1.6002679 -0.2219 -0.439"/>
 	</xacro:sensor_d415_left>
 	<xacro:sensor_d415_right parent="base_link" name="$(arg camera_name_right)" use_nominal_extrinsics="$(arg use_nominal_extrinsics)">
-		<origin xyz="0.42 -0.11026 -0.03433" rpy="-1.6002679 0.2855055 -6.177199343"/>
+		<origin xyz="0.415 -0.0928 0.025233" rpy="1.5413221 -0.3219 0.439"/>
 	</xacro:sensor_d415_right>
 	<xacro:gazebo_d435 camera_name="$(arg camera_name_left)" reference_link="$(arg camera_name_left)_link" topics_ns="/" depth_optical_frame="$(arg camera_name_left)_depth_optical_frame" color_optical_frame="$(arg camera_name_left)_color_optical_frame" infrared1_optical_frame="$(arg camera_name_left)_infrared1_optical_frame" infrared2_optical_frame="$(arg camera_name_left)_infrared2_optical_frame"/>
