Commit message: minor changes to launch files

File: src/seven_robot_description/urdf/sr-300.urdf.xacro (robot description, xacro)
@@ -58,16 +58,16 @@
 	<xacro:property name="wheel_radius" value="0.08641"/>
 	<link name="base_link">
-    <visual>
-			<origin rpy="${PI} 0 0" xyz="0 0 0"/>
-			<geometry>
-				<mesh filename="package://seven_robot_description/meshes/sr300_chasis.dae"/>
-			</geometry>
-		</visual>
-		<collision>
-		 <origin xyz="0 0 0.204528" rpy="0 0 0"/>
-		 <geometry>
-			<box size="${base_size_x} ${base_size_y} 0.47057"/>
-		 </geometry>
-		</collision>
+    	<visual>
+		<origin rpy="${PI} 0 0" xyz="0 0 0"/>
+		<geometry>
+			<mesh filename="package://seven_robot_description/meshes/sr300_chasis.dae"/>
+		</geometry>
+	</visual>
+	<collision>
+	 <origin xyz="0 0 0.204528" rpy="0 0 0"/>
+	 <geometry>
+	   <box size="${base_size_x} ${base_size_y} 0.47057"/>
+	 </geometry>
+	</collision>
 	</link>
 	<link name="base_footprint"/>
@@ -78,9 +78,9 @@
 	</joint>
 	<link name="inertial_link">
-		<inertial>
-			<mass value="47000.4"/>
-			<origin xyz="-0.01687 -0.00816 0.37647" rpy="0 0 0"/>
-			<inertia ixx="12585" ixy="-15.56" ixz="536.42" iyx="-15.56" iyy="806.894" iyz="-130.895" izx="-536.424" izy="-130.895" izz="5242.6"/>
-		</inertial>
+	 <inertial>
+	   <mass value="47000.4"/>
+	   <origin xyz="-0.01687 -0.00816 0.37647" rpy="0 0 0"/>
+	   <inertia ixx="12585" ixy="-15.56" ixz="536.42" iyx="-15.56" iyy="806.894" iyz="-130.895" izx="-536.424" izy="-130.895" izz="5242.6"/>
+	 </inertial>
 	</link>
 	<joint name="inertial_joint" type="fixed">
@@ -100,5 +100,5 @@
 	  <robotNamespace>/</robotNamespace>
 	  <updateRate>50.0</updateRate>
-    <bodyName>imu_link</bodyName>
+    	  <bodyName>imu_link</bodyName>
 	  <topicName>imu</topicName>
 	  <accelDrift>0.005 0.005 0.005</accelDrift>
@@ -111,20 +111,20 @@
   </gazebo>
 	<joint name="sick_base_joint" type="fixed">
-		<origin xyz="0.375 -0.219 0.13329" rpy="${PI} 0 -${PI/4}"/>
-   <parent link="base_link"/>
+	 <origin xyz="0.375 -0.219 0.13329" rpy="${PI} 0 -${PI/4}"/>
+   	 <parent link="base_link"/>
 	 <child link="sick_mount_link"/>
 	</joint>
 	<xacro:pu_wheel_sr300 prefix="Right">
-		<origin xyz="0.025 0.1918 0.02342" rpy="-${PI/2} 0 0"/>
+	 <origin xyz="0.025 0.1918 0.02342" rpy="-${PI/2} 0 0"/>
 	</xacro:pu_wheel_sr300>
 	<xacro:pu_wheel_sr300 prefix="Left">
-		<origin xyz="0.025 -0.1958 0.02291" rpy="${PI/2} 0 0"/>
+	 <origin xyz="0.025 -0.1958 0.02291" rpy="${PI/2} 0 0"/>
 	</xacro:pu_wheel_sr300>
 	<xacro:sick_lms_1xx name="sick" ros_topic="scan"/>
 	<xacro:sensor_d415_left parent="base_link" name="$(arg camera_name_left)" use_nominal_extrinsics="$(arg use_nominal_extrinsics)">
-		<origin xyz="0.415 0.1178 0.022233" rpy="1.6002679 -0.2219 -0.439"/>
+	 <origin xyz="0.415 0.1178 0.022233" rpy="1.6002679 -0.2219 -0.439"/>
 	</xacro:sensor_d415_left>
 	<xacro:sensor_d415_right parent="base_link" name="$(arg camera_name_right)" use_nominal_extrinsics="$(arg use_nominal_extrinsics)">
-		<origin xyz="0.415 -0.0928 0.025233" rpy="1.5413221 -0.3219 0.439"/>
+	 <origin xyz="0.415 -0.0928 0.025233" rpy="1.5413221 -0.3219 0.439"/>
 	</xacro:sensor_d415_right>
 	<xacro:gazebo_d435 camera_name="$(arg camera_name_left)" reference_link="$(arg camera_name_left)_link" topics_ns="/" depth_optical_frame="$(arg camera_name_left)_depth_optical_frame" color_optical_frame="$(arg camera_name_left)_color_optical_frame" infrared1_optical_frame="$(arg camera_name_left)_infrared1_optical_frame" infrared2_optical_frame="$(arg camera_name_left)_infrared2_optical_frame"/>

Commit message: added refined_path (corrections) 	modified:   env_loader_udooqdl.sh 	modified:   src/seven_bt_navigator 	modified:   src/seven_bt_plugins 	modified:   src/seven_mission_handler 	modified:   src/seven_robot_base/config/realsense_depth_filter.json 	modified:   src/seven_robot_base/launch/base.launch 	modified:   src/seven_robot_base/launch/dual_realsense.launch 	modified:   src/seven_robot_base/launch/top_level.launch 	modified:   src/seven_robot_base/params/robotParams.yaml 	modified:   src/seven_robot_base/params/system.yaml 	modified:   src/seven_robot_base/scripts/pyrealsense_mod.py 	modified:   src/seven_robot_description/launch/description.launch 	modified:   src/seven_robot_description/urdf/sr-300.urdf.xacro 	modified:   src/seven_robot_localization/launch/seven_robot_localization.launch 	modified:   src/seven_robot_localization/launch/sick_driver.launch 	modified:   src/seven_robot_localization/params/amcl.yaml 	modified:   src/seven_robot_localization/params/ekf.yaml 	modified:   src/seven_robot_utils 	modified:   src/seven_robotics_msgs 	modified:   src/uavcan_ros_bridge 	modified:   src/closest_point_of_approach (modified content) 	modified:   src/seven_bt_navigator (modified content) 	modified:   src/seven_bt_plugins (modified content, untracked content) 	modified:   src/seven_depth_utils (modified content, untracked content) 	modified:   src/seven_mission_handler (modified content) 	modified:   src/seven_path_smoother (modified content) 	modified:   src/seven_robot_navigation (modified content, untracked content) 	modified:   src/seven_robot_perception (modified content) 	modified:   src/seven_robot_utils (modified content) 	modified:   src/seven_robotics_msgs (modified content, untracked content) 	modified:   src/teb_local_planner (modified content, untracked content)

File: src/seven_robot_description/urdf/sr-300.urdf.xacro (robot description, xacro)
@@ -110,8 +110,8 @@
   	</gazebo>
 	<xacro:sensor_d415 parent="base_link" name="$(arg camera_name_left)" use_nominal_extrinsics="$(arg use_nominal_extrinsics)">
-	 <origin xyz="0.415 0.1178 0.022233" rpy="-1.6002679 -0.2219 -0.439"/>
+	 <origin xyz="0.3975 0.09958 0.019233" rpy="-1.5413221 -0.26 -0.439"/>
 	</xacro:sensor_d415>
 	<xacro:sensor_d415 parent="base_link" name="$(arg camera_name_right)" use_nominal_extrinsics="$(arg use_nominal_extrinsics)">
-	 <origin xyz="0.415 -0.0928 0.025233" rpy="-1.5413221 -0.3219 0.439"/>
+	 <origin xyz="0.4125 -0.1178 0.021233" rpy="-1.6013221 -0.26 0.439"/>
 	</xacro:sensor_d415>
 	<joint name="sick_base_joint" type="fixed">
